File: PCB/e'sPad/e'sPad.kicad_pcb (KiCad board)
At the start: 2 copper layers, 10 parts, among them SW1 SW_Push, SW2 SW_Push, SW3 SW_Push, SW4 SW_Push, SW5 SW_Push, SW6 SW_Push, SW7 RotaryEncoder, U1 XIAO-RP2040-DIP

Commit message: finished v1
Parts:
- added G***: LOGO, Battery:zelda_logo_footprint7, F.Cu at (164.3, 40.5)
- moved SW7 68.8 mm to (111.7, 38.0)
- moved U1 66.3 mm to (137.6, 41.0)
- moved D1 62.6 mm to (154.8, 34.8)
- moved D2 58.2 mm to (155.4, 44.4)
- moved SW1 13.5 mm to (121.6, 56.8)
- moved SW3 11.2 mm to (140.7, 56.8)
- moved SW2 11.0 mm to (121.6, 75.9)
- moved SW5 9.98 mm to (159.7, 56.8)
- moved SW4 7.94 mm to (140.7, 75.9)
- moved SW6 6.08 mm to (159.7, 75.9)
Routing:
- net GND: track 0.00 -> 176.6 mm
- net Net-(U1-GPIO7/SCL): track 0.00 -> 62.1 mm
- net Net-(U1-GPIO3/MOSI): track 0.00 -> 49.9 mm
- net Net-(U1-GPIO0/TX): track 0.00 -> 44.2 mm, vias 0 -> 3
- net Net-(U1-GPIO4/MISO): track 0.00 -> 41.4 mm
- net Net-(U1-GPIO1/RX): track 0.00 -> 34.5 mm
- net Net-(D1-DIN): track 0.00 -> 31.2 mm, vias 0 -> 1
- net Net-(U1-GPIO27/ADC1/A1): track 0.00 -> 26.8 mm
- net Net-(U1-GPIO2/SCK): track 0.00 -> 22.9 mm, vias 0 -> 1
- net +5V: track 0.00 -> 22.3 mm
- net Net-(U1-GPIO28/ADC2/A2): track 0.00 -> 19.1 mm
- net Net-(D1-DOUT): track 0.00 -> 13.0 mm
Other:
- board outline added: 61.9 x 62.7 mm
- board text added: "E's Custom Macropad"
- board text added: "XIAO HERE"
